Commit message: 更改了urdf质量，可以完成站立和行走，接下来先做减法

File: resources/robots/mini_cheetah/urdf/mini_cheetah.urdf (robot description, URDF)
Before this commit: robot mini_cheetah, 19 links, 18 joints
Links:
- link FL_thigh: mass 0.634 -> 2.136
- link FR_thigh: mass 0.634 -> 2.136
- link RL_thigh: mass 0.634 -> 2.136
- link RR_thigh: mass 0.634 -> 2.136
- link base: mass 3.3 -> 3.8
